Commit message: something is in gazebo

File: src/arm_full/config/panda.ros2_control.xacro (robot description, xacro)
@@ -1,16 +1,16 @@
 <?xml version="1.0"?>
 <robot xmlns:xacro="http://www.ros.org/wiki/xacro">
-    <xacro:macro name="panda_ros2_control" params="name initial_positions_file ros2_control_hardware_type">
+    <xacro:macro name="panda_ros2_control_ext" params="sys_name initial_positions_file ros2_control_hardware_type">
         <xacro:property name="initial_positions" value="${xacro.load_yaml(initial_positions_file)['initial_positions']}"/>
-        <ros2_control name="${name}" type="system">
+        <ros2_control name="${sys_name}" type="system">
             <hardware>
-                <xacro:if value="${ros2_control_hardware_type == 'mock_components'}">
-                    <plugin>mock_components/GenericSystem</plugin>
-                </xacro:if>
-                <xacro:if value="${ros2_control_hardware_type == 'isaac'}">
-                    <plugin>topic_based_ros2_control/TopicBasedSystem</plugin>
-                    <param name="joint_commands_topic">/isaac_joint_commands</param>
-                    <param name="joint_states_topic">/isaac_joint_states</param>
-                </xacro:if>
+              <!-- If launched with: ros2_control_hardware_type:=gz -->
+              <xacro:if value="${ros2_control_hardware_type == 'gz'}">
+                <plugin>gz_ros2_control/GazeboSystem</plugin>
+              </xacro:if>
+              <!-- Otherwise stay on fake hardware -->
+              <xacro:unless value="${ros2_control_hardware_type == 'gz'}">
+                <plugin>mock_components/GenericSystem</plugin>
+              </xacro:unless>
             </hardware>
             <joint name="panda_joint1">

File: src/arm_full/config/panda.urdf.xacro (robot description, xacro)
@@ -1,12 +1,14 @@
 <?xml version="1.0"?>
 <robot xmlns:xacro="http://www.ros.org/wiki/xacro" name="panda">
-    <xacro:arg name="initial_positions_file" default="initial_positions.yaml" />
+    <xacro:arg name="initial_positions_file" default="$(find arm_full)/config/initial_positions.yaml" />
     <xacro:arg name="ros2_control_hardware_type" default="mock_components" />
     <!-- Import panda urdf file -->
     <xacro:include filename="$(find arm_full)/urdf/panda.urdf.xacro" />
     <!-- Import panda ros2_control description -->
-    <xacro:include filename="panda.ros2_control.xacro" />
-    <xacro:include filename="panda_hand.ros2_control.xacro" />
-    <xacro:panda_ros2_control name="PandaFakeSystem" initial_positions_file="$(arg initial_positions_file)" ros2_control_hardware_type="$(arg ros2_control_hardware_type)"/>
+    <xacro:include filename="$(find arm_full)/config/panda.ros2_control.xacro" />
+    <xacro:include filename="$(find arm_full)/config/panda_hand.ros2_control.xacro" />
+    <xacro:panda_ros2_control_ext sys_name="PandaSystem"
+                            initial_positions_file="$(arg initial_positions_file)"
+                            ros2_control_hardware_type="$(arg ros2_control_hardware_type)"/>
     <xacro:panda_hand_ros2_control name="PandaHandFakeSystem" ros2_control_hardware_type="$(arg ros2_control_hardware_type)"/>
 </robot>

File: src/arm_full/config/panda_hand.ros2_control.xacro (robot description, xacro)
@@ -4,12 +4,10 @@
         <ros2_control name="${name}" type="system">
             <hardware>
-                <xacro:if value="${ros2_control_hardware_type == 'mock_components'}">
-                    <plugin>mock_components/GenericSystem</plugin>
-                </xacro:if>
-                <xacro:if value="${ros2_control_hardware_type == 'isaac'}">
-                    <plugin>topic_based_ros2_control/TopicBasedSystem</plugin>
-                    <param name="joint_commands_topic">/isaac_joint_commands</param>
-                    <param name="joint_states_topic">/isaac_joint_states</param>
-                </xacro:if>
+            <xacro:if value="${ros2_control_hardware_type == 'gz'}">
+                <plugin>gz_ros2_control/GazeboSystem</plugin>
+            </xacro:if>
+            <xacro:unless value="${ros2_control_hardware_type == 'gz'}">
+                <plugin>mock_components/GenericSystem</plugin>
+            </xacro:unless>
             </hardware>
             <joint name="panda_finger_joint1">

Commit message: wokring in gazebo with sim time false paramters

File: src/arm_full/config/panda.ros2_control.xacro (robot description, xacro)
@@ -5,12 +5,11 @@
         <ros2_control name="${sys_name}" type="system">
             <hardware>
-              <!-- If launched with: ros2_control_hardware_type:=gz -->
-              <xacro:if value="${ros2_control_hardware_type == 'gz'}">
-                <plugin>gz_ros2_control/GazeboSystem</plugin>
-              </xacro:if>
-              <!-- Otherwise stay on fake hardware -->
-              <xacro:unless value="${ros2_control_hardware_type == 'gz'}">
-                <plugin>mock_components/GenericSystem</plugin>
-              </xacro:unless>
+                <!-- If launched with: ros2_control_hardware_type:=gz -->
+                <xacro:if value="${ros2_control_hardware_type == 'gz'}">
+                  <plugin>gz_ros2_control/GazeboSimSystem</plugin>
+                </xacro:if>
+                <xacro:unless value="${ros2_control_hardware_type == 'gz'}">
+                  <plugin>mock_components/GenericSystem</plugin>
+                </xacro:unless>
             </hardware>
             <joint name="panda_joint1">

File: src/arm_full/config/panda.urdf.xacro (robot description, xacro)
@@ -12,3 +12,12 @@
                             ros2_control_hardware_type="$(arg ros2_control_hardware_type)"/>
     <xacro:panda_hand_ros2_control name="PandaHandFakeSystem" ros2_control_hardware_type="$(arg ros2_control_hardware_type)"/>
+    <gazebo>
+        <plugin filename="libgz_ros2_control-system.so"
+                name="gz_ros2_control::GazeboSimROS2ControlPlugin">
+            <!-- point to your controllers yaml -->
+            <parameters>$(find arm_full)/config/ros2_controllers.yaml</parameters>
+            <!-- hold joints at their commanded positions even when idle -->
+            <hold_joints>true</hold_joints>
+        </plugin>
+    </gazebo>
 </robot>

File: src/arm_full/config/panda_hand.ros2_control.xacro (robot description, xacro)
@@ -4,10 +4,11 @@
         <ros2_control name="${name}" type="system">
             <hardware>
-            <xacro:if value="${ros2_control_hardware_type == 'gz'}">
-                <plugin>gz_ros2_control/GazeboSystem</plugin>
-            </xacro:if>
-            <xacro:unless value="${ros2_control_hardware_type == 'gz'}">
+                <!-- If launched with: ros2_control_hardware_type:=gz -->
+                <xacro:if value="${ros2_control_hardware_type == 'gz'}">
+                <plugin>gz_ros2_control/GazeboSimSystem</plugin>
+                </xacro:if>
+                <xacro:unless value="${ros2_control_hardware_type == 'gz'}">
                 <plugin>mock_components/GenericSystem</plugin>
-            </xacro:unless>
+                </xacro:unless>
             </hardware>
             <joint name="panda_finger_joint1">

File: src/arm_full/urdf/panda.urdf.xacro (robot description, xacro)
@@ -5,4 +5,9 @@
 <!-- =================================================================================== -->
 <robot name="panda" xmlns:xacro="http://www.ros.org/wiki/xacro">
+    <link name="world"/>
+    <joint name="world_to_base" type="fixed">
+        <parent link="world"/>
+        <child  link="panda_link0"/>
+    </joint>
     <link name="panda_link0">
         <visual>
