Commit message: working griiper and everything in gazebo

File: src/arm_full/config/panda_hand.ros2_control.xacro (robot description, xacro)
@@ -13,19 +13,16 @@
             </hardware>
             <joint name="panda_finger_joint1">
-                <command_interface name="position" />
-                <state_interface name="position">
-                  <param name="initial_value">0.0</param>
-                </state_interface>
-                <state_interface name="velocity">
-                    <param name="initial_value">0.0</param>
-                </state_interface>
+            <command_interface name="position" />
+            <state_interface name="position">
+                <param name="initial_value">0.035</param>
+            </state_interface>
+            <state_interface name="velocity"><param name="initial_value">0.0</param></state_interface>
             </joint>
             <joint name="panda_finger_joint2">
-                <state_interface name="position">
-                  <param name="initial_value">0.0</param>
-                </state_interface>
-                <state_interface name="velocity">
-                    <param name="initial_value">0.0</param>
-                </state_interface>
+            <command_interface name="position" />
+            <state_interface name="position">
+                <param name="initial_value">0.035</param>
+            </state_interface>
+            <state_interface name="velocity"><param name="initial_value">0.0</param></state_interface>
             </joint>
         </ros2_control>

File: src/arm_full/urdf/panda.urdf.xacro (robot description, xacro)
@@ -288,5 +288,5 @@
         <axis xyz="0 -1 0" />
         <limit effort="20" lower="0.0" upper="0.04" velocity="0.2" />
-        <mimic joint="panda_finger_joint1" />
+        <!-- <mimic joint="panda_finger_joint1" /> -->
         <dynamics damping="0.3" />
     </joint>
