Commit message: added gazebo

File: src/moveit_resources/panda_description/urdf/panda.urdf.xacro (robot description, xacro)
@@ -5,4 +5,9 @@
 <!-- =================================================================================== -->
 <robot name="panda" xmlns:xacro="http://www.ros.org/wiki/xacro">
+    <link name="world"/>
+    <joint name="world_to_base" type="fixed">
+        <parent link="world"/>
+        <child  link="panda_link0"/>
+    </joint>
     <link name="panda_link0">
         <visual>
@@ -283,5 +288,5 @@
         <axis xyz="0 -1 0" />
         <limit effort="20" lower="0.0" upper="0.04" velocity="0.2" />
-        <mimic joint="panda_finger_joint1" />
+        <!-- <mimic joint="panda_finger_joint1" /> -->
         <dynamics damping="0.3" />
     </joint>

File: src/moveit_resources/panda_moveit_config/config/panda.ros2_control.xacro (robot description, xacro)
@@ -5,4 +5,7 @@
         <ros2_control name="${name}" type="system">
             <hardware>
+                <xacro:if value="${ros2_control_hardware_type == 'gz'}">
+                    <plugin>gz_ros2_control/GazeboSimSystem</plugin>
+                </xacro:if>
                 <xacro:if value="${ros2_control_hardware_type == 'mock_components'}">
                     <plugin>mock_components/GenericSystem</plugin>

File: src/moveit_resources/panda_moveit_config/config/panda.urdf.xacro (robot description, xacro)
@@ -8,5 +8,18 @@
     <xacro:include filename="panda.ros2_control.xacro" />
     <xacro:include filename="panda_hand.ros2_control.xacro" />
-    <xacro:panda_ros2_control name="PandaFakeSystem" initial_positions_file="$(arg initial_positions_file)" ros2_control_hardware_type="$(arg ros2_control_hardware_type)"/>
-    <xacro:panda_hand_ros2_control name="PandaHandFakeSystem" ros2_control_hardware_type="$(arg ros2_control_hardware_type)"/>
+    <xacro:panda_ros2_control name="PandaSystem"
+                            initial_positions_file="$(arg initial_positions_file)"
+                            ros2_control_hardware_type="$(arg ros2_control_hardware_type)"/>
+    <xacro:panda_hand_ros2_control
+        name="PandaHandFakeSystem"
+        ros2_control_hardware_type="$(arg ros2_control_hardware_type)"/>
+    <gazebo>
+        <plugin filename="libgz_ros2_control-system.so"
+                name="gz_ros2_control::GazeboSimROS2ControlPlugin">
+            <!-- point to your controllers yaml -->
+            <parameters>$(find moveit_resources_panda_moveit_config)/config/ros2_controllers.yaml</parameters>
+            <!-- hold joints at their commanded positions even when idle -->
+            <hold_joints>true</hold_joints>
+        </plugin>
+    </gazebo>
 </robot>

File: src/moveit_resources/panda_moveit_config/config/panda_hand.ros2_control.xacro (robot description, xacro)
@@ -4,4 +4,7 @@
         <ros2_control name="${name}" type="system">
             <hardware>
+                <xacro:if value="${ros2_control_hardware_type == 'gz'}">
+                    <plugin>gz_ros2_control/GazeboSimSystem</plugin>
+                </xacro:if>
                 <xacro:if value="${ros2_control_hardware_type == 'mock_components'}">
                     <plugin>mock_components/GenericSystem</plugin>
@@ -23,4 +26,5 @@
             </joint>
             <joint name="panda_finger_joint2">
+                <command_interface name="position" />
                 <state_interface name="position">
                   <param name="initial_value">0.0</param>
